File: KiCad/WaterValveX4.kicad_pcb (KiCad board)
At the start: 2 copper layers, 63.2 x 39.1 mm, 50 parts, among them J1 Conn_01x04_Male, J2 Barrel_Jack, J3 Conn_01x03_Male, J4 Conn_01x01_Male, J5 Conn_01x04_Male, J6 Screw_Terminal_01x03, J7 Screw_Terminal_01x03, J8 Screw_Terminal_01x03, J9 Screw_Terminal_01x02, Q1 IRLML2502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

Commit message: Change to use ESP32 C6 THT
Parts:
- D11: footprint LED_SMD:LED_0805_2012Metric_Pad1.15x1.40mm_HandSolder -> LED_THT:LED_D5.0mm; moved to B.Cu
- U2: value SeedStudio XIAO ESP32 C3 v1 -> XIAO-ESP32-C6; footprint LOCAL1:XIAO_ESP32C3_THT -> LOCAL1:XIAO-ESP32-C6-DIP
- moved U2 13.6 mm to (162.6, 109.8)
- moved D11 1.49 mm to (177.3, 90.5)
- moved R4 1.09 mm to (177.0, 119.5)
- moved R5 0.54 mm to (174.5, 119.5)
Connections:
- R6 pad 1: /GPIO1 -> /GPIO3
- R8 pad 1: /GPIO5 -> /GPIO4
- R9 pad 1: /GPIO3 -> /GPIO5
- U2 pad 2: /GPIO1 -> /GPIO3
- U2 pad 3: /GPIO5 -> /GPIO4
- U2 pad 4: /GPIO3 -> /GPIO5
Routing:
- net +5V: track 85.6 -> 71.0 mm
- net /SDA: track 36.9 -> 28.9 mm, vias 0 -> 1
- net /GPIO5: track 4.27 -> 9.85 mm
- net +3V3: track 86.2 -> 81.3 mm
- net /GPIO4: track 0.00 -> 4.58 mm
- net /PwrIn: track 55.8 -> 60.1 mm
- net +VSW: track 56.3 -> 52.3 mm
- net /GPIO1: track 3.44 -> 0.00 mm
- net /SCL: track 27.9 -> 25.4 mm
- net Net-(D1-K): track 10.3 -> 12.7 mm, vias 0 -> 1
- net /GPIO3: track 5.73 -> 3.75 mm
- net /GPIO2: track 30.5 -> 29.0 mm
- net Net-(D11-K): track 2.05 -> 2.96 mm
- net Net-(D3-K): track 3.12 -> 3.90 mm
- net /RX: track 3.25 -> 3.86 mm
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Other:
- board text added: "(C) 2025 Hans Rune Bue <email@hansrune.net>"
- board text added: "WaterValveX4 - Rev 3.0"
- board text removed: "(C) 2023 Hans Rune Bue <email@hansrune.net>"
- board text removed: "WaterValveX4 - Rev 2.0.1"

Commit message: Optimized layout - passes most DRC checks
Parts:
- added D13: LED, LED_SMD:LED_0805_2012Metric_Pad1.15x1.40mm_HandSolder, F.Cu at (174.8, 88.5)
- added D14: LED, LED_THT:LED_D3.0mm, B.Cu at (166.1, 95.9)
- added D15: LED, LED_THT:LED_D3.0mm, B.Cu at (183.2, 115.0)
- added D16: LED, LED_THT:LED_D3.0mm, B.Cu at (183.2, 109.7)
- added D17: LED, LED_THT:LED_D3.0mm, B.Cu at (183.5, 104.2)
- added D18: LED, LED_THT:LED_D3.0mm, B.Cu at (183.5, 98.2)
- D10, D3, D5, D8: moved to F.Cu
- D11: footprint LED_THT:LED_D5.0mm -> LED_THT:LED_D3.0mm
- D12, D4, D6, D9: footprint Diode_THT:D_DO-41_SOD81_P3.81mm_Vertical_KathodeUp -> Diode_THT:D_DO-41_SOD81_P2.54mm_Vertical_KathodeUp
- moved D12 4.59 mm to (187.8, 97.5), turned to -90 degrees
- moved D10 3.81 mm to (184.8, 98.5), turned to 0 degrees
- moved D9 3.66 mm to (187.8, 103.5), turned to -90 degrees
- moved R15 3.54 mm to (180.8, 97.0), turned to 0 degrees
- moved D4 3.42 mm to (187.8, 114.5), turned to -90 degrees
- moved D6 3.35 mm to (187.8, 109.0), turned to -90 degrees
- moved D3 3.24 mm to (184.5, 115.0), turned to 0 degrees
- moved D8 3.14 mm to (184.8, 104.2), turned to 0 degrees
- moved D5 2.89 mm to (184.5, 109.7), turned to 0 degrees
- moved Q1 2.77 mm to (179.2, 115.8)
- moved R6 2.45 mm to (174.0, 115.8)
- moved R13 2.41 mm to (180.8, 102.5), turned to 0 degrees
- moved D11 2.35 mm to (176.0, 88.5)
- moved R11 2.24 mm to (174.5, 98.2), turned to 180 degrees
- moved R12 2.21 mm to (173.5, 92.8)
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Connections:
- net /GPIO10 renamed /D10
- net /GPIO3 renamed /D1
- net /GPIO4 renamed /D2
- net /GPIO5 renamed /D3
- net /GPIO8 renamed /D8
Routing:
- net GND: track 0.00 -> 23.8 mm, vias 0 -> 4
- net +VSW: track 52.3 -> 64.8 mm
- net /Relay4: track 18.3 -> 29.9 mm
- net Net-(Q4-G): track 2.33 -> 9.92 mm, vias 0 -> 2
- net /GPIO2: track 29.0 -> 35.5 mm, vias 1 -> 2
- net +3V3: track 81.3 -> 87.4 mm
- net /D3: track 9.85 -> 5.71 mm
- net /SDA: track 28.9 -> 32.9 mm, vias 1 -> 0
- net /Relay1: track 17.8 -> 21.3 mm
- net /SCL: track 25.4 -> 28.0 mm
- net /D8: track 21.5 -> 24.0 mm
- net /PwrIn: track 60.1 -> 62.5 mm
- net Net-(D1-K): track 12.7 -> 14.5 mm
- net Net-(D1-A): track 10.8 -> 12.5 mm, vias 0 -> 1
- net Net-(Q3-G): track 2.35 -> 3.82 mm
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